Commit message: feat: add new end-effector frame at the tip of the gripper

File: urdf/yumi_full.urdf (robot description, URDF)
Before this commit: robot yumi, 22 links, 21 joints
Links:
- added link gripper_l_tip
- added link gripper_r_tip
Joints:
- added joint gripper_l_tip_fixed: type fixed, parent gripper_l_base, child gripper_l_tip, origin xyz=0 0 0.13 rpy=0 0 3.14159265359
- added joint gripper_r_tip_fixed: type fixed, parent gripper_r_base, child gripper_r_tip, origin xyz=0 0 0.13 rpy=0 0 3.14159265359

File: urdf/yumi_left.urdf (robot description, URDF)
Before this commit: robot yumi, 12 links, 11 joints
Links:
- added link gripper_l_tip
Joints:
- added joint gripper_l_tip_fixed: type fixed, parent gripper_l_base, child gripper_l_tip, origin xyz=0 0 0.13 rpy=0 0 3.14159265359

File: urdf/yumi_right.urdf (robot description, URDF)
Before this commit: robot yumi, 12 links, 11 joints
Links:
- added link gripper_r_tip
Joints:
- added joint gripper_r_tip_fixed: type fixed, parent gripper_r_base, child gripper_r_tip, origin xyz=0 0 0.13 rpy=0 0 3.14159265359
